File: voodoo_1.kicad_pcb (KiCad board)
At the start: 2 copper layers, 60 x 42 mm, 41 parts, among them Q1 2N2222, Q2 2N2222, U1 LM308

Commit message: ベタを修正
Other:
- board size 60 x 42 mm -> 59 x 42 mm
Changed lines of the file:
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@@
 	)
 	(gr_rect
-		(start 41 77)
+		(start 42 77)
 		(end 101 119)
 		(stroke
@@
 		(polygon
 			(pts
-				(xy 41 76.3) (xy 101.7 76.7) (xy 102.4 119.8) (xy 39.3 119.7) (xy 41 76.2)
+				(xy 42 114) (xy 42 82) (xy 47 77) (xy 96 77) (xy 101 82) (xy 101 114) (xy 96 119) (xy 47 119)
 			)
 		)
